Commit message: fixed issues

File: description/urdf/bluerov2.urdf (robot description, URDF)
Before this commit: robot ceto_description/description, 8 links, 7 joints
Links:
- added link camera_mount_link, mass 0.0001
- link base_link: geometry collision box size=0.457 0.338 0.065; visual mesh filename=package://ceto_description/description/meshes/bluerov2.dae scale=0.025 0.025 0.025
- link thruster1: geometry visual mesh filename=package://ceto_description/description/meshes/ccw_prop.dae
- link thruster2: geometry visual mesh filename=package://ceto_description/description/meshes/ccw_prop.dae
- link thruster3: geometry visual mesh filename=package://ceto_description/description/meshes/ccw_prop.dae
- link thruster4: geometry visual mesh filename=package://ceto_description/description/meshes/ccw_prop.dae
- link thruster5: geometry visual mesh filename=package://ceto_description/description/meshes/ccw_prop.dae
- link thruster6: geometry visual mesh filename=package://ceto_description/description/meshes/ccw_prop.dae
Joints:
- added joint camera_mount_joint: type fixed, parent base_link, child camera_mount_link, origin xyz=0.19 0 0.067 rpy=0 0 0
