Commit message: added bluerov model for testing, changed name and config

File: urdf/robot.urdf.xacro (robot description, xacro)
@@ -1,415 +1,170 @@
-<?xml version="1.0" ?>
-<robot name="auv" xmlns:xacro="http://www.ros.org/wiki/xacro">
-  <!-- <xacro:include filename="$(find sauvc_sim)/urdf/thrusters.xacro"/> -->
-  <xacro:include filename="$(find sauvc_sim)/urdf/sensors.xacro"/>
-  <xacro:include filename="$(find sauvc_sim)/urdf/plugins.xacro"/>
+<?xml version="1.0"?>
+<robot name="ceto">
+  <!-- Base Link -->
   <link name="base_link">
-    <!-- Inertial properties -->
     <inertial>
-      <origin xyz="0 0 -0.59" rpy="0 0 0"/>
-      <mass value="1862.87"/>
-      <inertia
-        ixx="525.39" ixy="1.44" ixz="33.41"
-        iyy="794.20" iyz="2.6"  izz="691.23"/>
+      <origin xyz="0.0 0.0 0.011" rpy="0 0 0"/>
+      <mass value="10.0"/>
+      <inertia ixx="0.099" ixy="0" ixz="0" iyy="0.178" iyz="0" izz="0.269"/>
     </inertial>
-    <!-- Visual mesh -->
     <visual>
       <origin xyz="0 0 0" rpy="0 0 0"/>
       <geometry>
-        <mesh filename="file://$(find sauvc_sim)/meshes/rexrov/RexROV_no_props.dae" scale="1 1 1"/>
+        <!-- Assuming a ROS package named 'ceto_description/description' exists -->
+        <mesh filename="file://$(find ceto_description)/meshes/bluerov2.dae" scale="0.025 0.025 0.025"/>
       </geometry>
     </visual>
-    <!-- Collision: bottom plate -->
     <collision>
-      <origin xyz="0 0 -0.75" rpy="0 0 0"/>
+      <origin xyz="0.0 0.0 0.06" rpy="0 0 0"/>
       <geometry>
-        <box size="2.56 1.50 0.10"/>
-      </geometry>
-    </collision>
-    <!-- Collision: top plate -->
-    <collision>
-      <origin xyz="0 0 0.60" rpy="0 0 0"/>
-      <geometry>
-        <box size="2.56 1.50 0.40"/>
-      </geometry>
-    </collision>
-    <!-- Collision: left side -->
-    <collision>
-      <origin xyz="-0.20 0.70 -0.15" rpy="0 0 0"/>
-      <geometry>
-        <box size="2.20 0.10 1.10"/>
-      </geometry>
-    </collision>
-    <!-- Collision: right side -->
-    <collision>
-      <origin xyz="0.20 -0.70 -0.15" rpy="0 0 0"/>
-      <geometry>
-        <box size="2.20 0.10 1.10"/>
+        <box size="0.457 0.338 0.065"/>
       </geometry>
     </collision>
   </link>
-<!-- Camera Link -->
+  <!-- Camera Mount Link -->
+  <link name="camera_mount_link">
+    <inertial>
+      <origin xyz="0 0 0" rpy="0 0 0"/>
+      <mass value="0.0001"/>
+      <inertia ixx="0.0001" ixy="0" ixz="0" iyy="0.0001" iyz="0" izz="0.0001"/>
+    </inertial>
+  </link>
+  <joint name="camera_mount_joint" type="fixed">
+    <origin xyz="0.19 0 0.067" rpy="0 0 0"/>
+    <parent link="base_link"/>
+    <child link="camera_mount_link"/>
+  </joint>
+  <!-- Camera Link -->
   <link name="camera_link">
-    <!-- Inertial -->
     <inertial>
-      <mass value="0.1"/>
-      <inertia
-        ixx="0.000166667" ixy="0.0" ixz="0.0"
-        iyy="0.000166667" iyz="0.0" izz="0.000166667"/>
+      <origin xyz="0 0 0" rpy="0 0 0"/>
+      <mass value="0.0001"/>
+      <inertia ixx="0.0001" ixy="0" ixz="0" iyy="0.0001" iyz="0" izz="0.0001"/>
     </inertial>
-    <!-- Collision -->
-    <collision>
+  </link>
+  <joint name="camera_joint" type="fixed">
+    <origin xyz="0 0 0" rpy="0 0 0"/>
+    <parent link="camera_mount_link"/>
+    <child link="camera_link"/>
+  </joint>
+  <!-- Thruster 1 -->
+  <link name="thruster1">
+    <inertial>
+      <origin xyz="0 0 0" rpy="0 0 0"/>
+      <mass value="0.002"/>
+      <inertia ixx="0.001" ixy="0" ixz="0" iyy="0.001" iyz="0" izz="0.001"/>
+    </inertial>
+    <visual>
+      <origin xyz="0 0 0" rpy="-1.571 0 0"/>
       <geometry>
-        <box size="0.1 0.1 0.1"/>
-      </geometry>
-    </collision>
-    <!-- Visual -->
-    <visual>
-      <geometry>
-        <box size="0.1 0.1 0.1"/>
+        <mesh filename="file://$(find ceto_description)/meshes/ccw_prop.dae"/>
       </geometry>
     </visual>
   </link>
-  <!-- Fixed joint between base_link and camera_link -->
-  <joint name="camera_joint" type="fixed">
-    <origin xyz="1.33 0 -0.74" rpy="0 0 0"/>
-    <parent link="base_link"/>
-    <child link="camera_link"/>
-  </joint>
-  <!-- Magnetometer Link -->
-  <link name="magnetometer_link">
-    <!-- <origin xyz="0 0 0" rpy="0 0 0"/> -->
-    <inertial>
-      <mass value="0.015"/>
-      <inertia
-        ixx="0.00001" ixy="0.0" ixz="0.0"
-        iyy="0.00001" iyz="0.0" izz="0.00001"/>
-    </inertial>
-  </link>
-    <joint name="magnetometer_joint" type="fixed">
-      <origin xyz='0 0 0' rpy='0 0 0'/>
-      <parent link="base_link" />
-      <child link="magnetometer_link" />
-    </joint>
-    <link name="imu_link">
-      <inertial>
-        <origin xyz="0 0 0" rpy="0 0 0"/>
-        <mass value="0.015"/>
-        <inertia ixx="0.00001" ixy="0.0" ixz="0.0" iyy="0.00001" iyz="0.0" izz="0.00001"/>
-      </inertial>
-    </link>
-    <joint name="imu_joint" type="fixed">
-      <origin xyz='0 0 0' rpy='0 0 0'/>
-      <parent link="base_link" />
-      <child link="imu_link" />
-    </joint>
-    <!-- <link name="dvl_link">
-      <origin xyz='-1.34 0 -0.75' rpy='0 0 -1.57'/>
-      <inertial>
-        <mass>3.5</mass>
-        <inertia>
-          <ixx>0.0195872</ixx>
-          <ixy>0</ixy>
-          <ixz>0</ixz>
-          <iyy>0.0195872</iyy>
-          <iyz>0</iyz>
-          <izz>0.0151357</izz>
-        </inertia>
-      </inertial>
-      <velocity_decay />
-      <gravity>1</gravity>
-      <velocity_decay />
-      <self_collide>0</self_collide>
-      <enable_wind>0</enable_wind>
-      <kinematic>0</kinematic>
-      <visual name="dvl_link_visual">
-        <origin xyz='0 0 0' rpy='0 0 3.14159'/>
-        <geometry>
-          <mesh>
-            <scale>1 1 1</scale>
-            <uri>model://meshes/nortek_dvl500_300/DVL500-300m.dae</uri>
-          </mesh>
-        </geometry>
-        <transparency>0</transparency>
-        <cast_shadows>1</cast_shadows>
-      </visual>
-      <collision name="dvl_link_collision">
-        <laser_retro>0</laser_retro>
-        <max_contacts>10</max_contacts>
-        <origin xyz='0 0 0' rpy='3.14159 0 0'/>
-        <geometry>
-          <cylinder>
-            <radius>0.093</radius>
-            <length>0.203</length>
-          </cylinder>
-        </geometry>
-        <surface>
-          <friction>
-            <ode>
-              <mu>1</mu>
-              <mu2>1</mu2>
-              <fdir1>0 0 0</fdir1>
-              <slip1>0</slip1>
-              <slip2>0</slip2>
-            </ode>
-            <torsional>
-              <coefficient>1</coefficient>
-              <patch_radius>0</patch_radius>
-              <surface_radius>0</surface_radius>
-              <use_patch_radius>1</use_patch_radius>
-              <ode>
-                <slip>0</slip>
-              </ode>
-            </torsional>
-          </friction>
-          <bounce>
-            <restitution_coefficient>0</restitution_coefficient>
-            <threshold>1e+06</threshold>
-          </bounce>
-          <contact>
-            <collide_without_contact>0</collide_without_contact>
-            <collide_without_contact_bitmask>1</collide_without_contact_bitmask>
-            <collide_bitmask>1</collide_bitmask>
-            <ode>
-              <soft_cfm>0</soft_cfm>
-              <soft_erp>0.2</soft_erp>
-              <kp>1e+13</kp>
-              <kd>1</kd>
-              <max_vel>0.01</max_vel>
-              <min_depth>0</min_depth>
-            </ode>
-            <bullet>
-              <split_impulse>1</split_impulse>
-              <split_impulse_penetration_threshold>-0.01</split_impulse_penetration_threshold>
-              <soft_cfm>0</soft_cfm>
-              <soft_erp>0.2</soft_erp>
-              <kp>1e+13</kp>
-              <kd>1</kd>
-            </bullet>
-          </contact>
-        </surface>
-      </collision>
-    </link>
-    <joint name="dvl_joint" type="fixed">
-      <origin xyz="-1.34 0 -0.75" rpy="0 0 -1.57"/>
-      <parent link="base_link" />
-      <child link="dvl_link" />
-    </joint>
--->
-  <!-- Thruster 1 -->
-  <link name="thruster1">
-     <!-- <origin xyz="-0.890895 0.334385 0.528822" rpy="0 -1.300794 -0.928689"/> -->
-    <inertial>
-      <mass value="0.001"/>
-      <inertia ixx="0.0005" ixy="0" ixz="0"
-              iyy="0.0005" iyz="0" izz="0.0005"/>
-    </inertial>
-    <visual>
-      <geometry>
-        <mesh filename="file://$(find sauvc_sim)/meshes/rexrov/prop.dae" scale="1 1 1"/>
-      </geometry>
-    </visual>
-    <collision>
-      <origin xyz="0 0 0" rpy="0 0 0"/>
-      <geometry>
-        <cylinder length="0.000001" radius="0.000001"/>
-      </geometry>
-    </collision>
-  </link>
-  <joint name="thruster1_joint" type="revolute">
-    <origin xyz="-0.890895 0.334385 0.528822" rpy="0 -1.300794 -0.928689"/>
+  <joint name="thruster1_joint" type="continuous">
+    <origin xyz="0.14 -0.092 0.0" rpy="-1.571 1.571 -0.785"/>
     <parent link="base_link"/>
     <child link="thruster1"/>
-    <axis xyz="1 0 0"/>
-    <limit effort="100" lower="-1000" upper="1000" velocity="100"/>
+    <axis xyz="0 0 -1"/>
   </joint>
   <!-- Thruster 2 -->
   <link name="thruster2">
-    <!-- <origin xyz="-0.890895 -0.334385 0.528822" rpy="0 -1.300794 0.928689"/> -->
     <inertial>
-      <mass value="0.001"/>
-      <inertia ixx="0.0005" ixy="0" ixz="0"
-              iyy="0.0005" iyz="0" izz="0.0005"/>
+      <origin xyz="0 0 0" rpy="0 0 0"/>
+      <mass value="0.002"/>
+      <inertia ixx="0.001" ixy="0" ixz="0" iyy="0.001" iyz="0" izz="0.001"/>
     </inertial>
     <visual>
+      <origin xyz="0 0 0" rpy="-1.571 0 0"/>
       <geometry>
-        <mesh filename="file://$(find sauvc_sim)/meshes/rexrov/prop.dae" scale="1 1 1"/>
+        <mesh filename="file://$(find ceto_description)/meshes/ccw_prop.dae"/>
       </geometry>
     </visual>
-    <collision>
-      <origin xyz="0 0 0" rpy="0 0 0"/>
-      <geometry>
-        <cylinder length="0.000001" radius="0.000001"/>
-      </geometry>
-    </collision>
   </link>
-  <joint name="thruster2_joint" type="revolute">
-    <origin xyz="-0.890895 -0.334385 0.528822" rpy="0 -1.300794 0.928689"/>
+  <joint name="thruster2_joint" type="continuous">
+    <origin xyz="0.14 0.092 0.0" rpy="-1.571 1.571 -2.356"/>
     <parent link="base_link"/>
     <child link="thruster2"/>
-    <axis xyz="1 0 0"/>
-    <limit effort="100" lower="-1000" upper="1000" velocity="100"/>
+    <axis xyz="0 0 -1"/>
   </joint>
   <!-- Thruster 3 -->
   <link name="thruster3">
-    <!-- <origin xyz="0.890895 0.334385 0.528822" rpy="0 -1.840798 0.928689"/> -->
     <inertial>
-      <mass value="0.001"/>
-      <inertia ixx="0.0005" ixy="0" ixz="0"
-              iyy="0.0005" iyz="0" izz="0.0005"/>
+      <origin xyz="0 0 0" rpy="0 0 0"/>
+      <mass value="0.002"/>
+      <inertia ixx="0.001" ixy="0" ixz="0" iyy="0.001" iyz="0" izz="0.001"/>
     </inertial>
     <visual>
+      <origin xyz="0 0 0" rpy="1.571 0 0"/>
       <geometry>
-        <mesh filename="file://$(find sauvc_sim)/meshes/rexrov/prop.dae" scale="1 1 1"/>
+        <mesh filename="file://$(find ceto_description)/meshes/ccw_prop.dae"/>
       </geometry>
     </visual>
-    <collision>
-      <origin xyz="0 0 0" rpy="0 0 0"/>
-      <geometry>
-        <cylinder length="0.000001" radius="0.000001"/>
-      </geometry>
-    </collision>
   </link>
-  <joint name="thruster3_joint" type="revolute">
-    <origin xyz="0.890895 0.334385 0.528822" rpy="0 -1.840798 0.928689"/>
+  <joint name="thruster3_joint" type="continuous">
+    <origin xyz="-0.15 -0.092 0.0" rpy="-1.571 1.571 0.785"/>
     <parent link="base_link"/>
     <child link="thruster3"/>
-    <axis xyz="1 0 0"/>
-    <limit effort="100" lower="-1000" upper="1000" velocity="100"/>
+    <axis xyz="0 0 -1"/>
   </joint>
   <!-- Thruster 4 -->
   <link name="thruster4">
-    <!-- <origin xyz="0.890895 -0.334385 0.528822" rpy="0 -1.300794 -0.928689"/> -->
     <inertial>
-      <mass value="0.001"/>
-      <inertia ixx="0.0005" ixy="0" ixz="0"
-              iyy="0.0005" iyz="0" izz="0.0005"/>
+      <origin xyz="0 0 0" rpy="0 0 0"/>
+      <mass value="0.002"/>
+      <inertia ixx="0.001" ixy="0" ixz="0" iyy="0.001" iyz="0" izz="0.001"/>
     </inertial>
     <visual>
+      <origin xyz="0 0 0" rpy="1.571 0 0"/>
       <geometry>
-        <mesh filename="file://$(find sauvc_sim)/meshes/rexrov/prop.dae" scale="1 1 1"/>
+        <mesh filename="file://$(find ceto_description)/meshes/ccw_prop.dae"/>
       </geometry>
     </visual>
-    <collision>
-      <origin xyz="0 0 0" rpy="0 0 0"/>
-      <geometry>
-        <cylinder length="0.000001" radius="0.000001"/>
-      </geometry>
-    </collision>
   </link>
-  <joint name="thruster4_joint" type="revolute">
-    <origin xyz="0.890895 -0.334385 0.528822" rpy="0 -1.300794 -0.928689"/>
+  <joint name="thruster4_joint" type="continuous">
+    <origin xyz="-0.15 0.092 0.0" rpy="-1.571 1.571 2.356"/>
     <parent link="base_link"/>
     <child link="thruster4"/>
-    <axis xyz="1 0 0"/>
-    <limit effort="100" lower="-1000" upper="1000" velocity="100"/>
+    <axis xyz="0 0 -1"/>
   </joint>
   <!-- Thruster 5 -->
   <link name="thruster5">
-    <!-- <origin xyz="-0.412125 0.505415 0.129" rpy="0 0 0.785398"/> -->
     <inertial>
-      <mass value="0.001"/>
-      <inertia ixx="0.0005" ixy="0" ixz="0"
-              iyy="0.0005" iyz="0" izz="0.0005"/>
+      <origin xyz="0 0 0" rpy="0 0 0"/>
+      <mass value="0.002"/>
+      <inertia ixx="0.001" ixy="0" ixz="0" iyy="0.001" iyz="0" izz="0.001"/>
     </inertial>
     <visual>
+      <origin xyz="0 0 0" rpy="-1.571 0 1.571"/>
       <geometry>
-        <mesh filename="file://$(find sauvc_sim)/meshes/rexrov/prop.dae" scale="1 1 1"/>
+        <mesh filename="file://$(find ceto_description)/meshes/ccw_prop.dae"/>
       </geometry>
     </visual>
-    <collision>
-      <origin xyz="0 0 0" rpy="0 0 0"/>
-      <geometry>
-        <cylinder length="0.000001" radius="0.000001"/>
-      </geometry>
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
Commit message: fixed

File: urdf/robot.urdf.xacro (robot description, xacro)
@@ -12,5 +12,5 @@
       <geometry>
         <!-- Assuming a ROS package named 'ceto_description/description' exists -->
-        <mesh filename="file://$(find ceto_description)/meshes/bluerov2.dae" scale="0.025 0.025 0.025"/>
+        <mesh filename="file://$(find ceto_description)/models/meshes/bluerov2.dae" scale="0.025 0.025 0.025"/>
       </geometry>
     </visual>
@@ -58,5 +58,5 @@
       <origin xyz="0 0 0" rpy="-1.571 0 0"/>
       <geometry>
-        <mesh filename="file://$(find ceto_description)/meshes/ccw_prop.dae"/>
+        <mesh filename="file://$(find ceto_description)/models/meshes/ccw_prop.dae"/>
       </geometry>
     </visual>
@@ -78,5 +78,5 @@
       <origin xyz="0 0 0" rpy="-1.571 0 0"/>
       <geometry>
-        <mesh filename="file://$(find ceto_description)/meshes/ccw_prop.dae"/>
+        <mesh filename="file://$(find ceto_description)/models/meshes/ccw_prop.dae"/>
       </geometry>
     </visual>
@@ -98,5 +98,5 @@
       <origin xyz="0 0 0" rpy="1.571 0 0"/>
       <geometry>
-        <mesh filename="file://$(find ceto_description)/meshes/ccw_prop.dae"/>
+        <mesh filename="file://$(find ceto_description)/models/meshes/ccw_prop.dae"/>
       </geometry>
     </visual>
@@ -118,5 +118,5 @@
       <origin xyz="0 0 0" rpy="1.571 0 0"/>
       <geometry>
-        <mesh filename="file://$(find ceto_description)/meshes/ccw_prop.dae"/>
+        <mesh filename="file://$(find ceto_description)/models/meshes/ccw_prop.dae"/>
       </geometry>
     </visual>
@@ -138,5 +138,5 @@
       <origin xyz="0 0 0" rpy="-1.571 0 1.571"/>
       <geometry>
-        <mesh filename="file://$(find ceto_description)/meshes/ccw_prop.dae"/>
+        <mesh filename="file://$(find ceto_description)/models/meshes/ccw_prop.dae"/>
       </geometry>
     </visual>
@@ -158,5 +158,5 @@
       <origin xyz="0 0 0" rpy="1.571 0 1.571"/>
       <geometry>
-        <mesh filename="file://$(find ceto_description)/meshes/ccw_prop.dae"/>
+        <mesh filename="file://$(find ceto_description)/models/meshes/ccw_prop.dae"/>
       </geometry>
     </visual>

Commit message: fixed urdf and added config

File: urdf/robot.urdf.xacro (robot description, xacro)
@@ -1,4 +1,11 @@
 <?xml version="1.0"?>
 <robot name="ceto">
+<!-- add a dummy root (no inertia) to satisfy KDL -->
+  <link name="root_link"/>
+  <joint name="root_to_base_fixed" type="fixed">
+    <parent link="root_link"/>
+    <child link="base_link"/>
+    <origin xyz="0 0 0" rpy="0 0 0"/>
+  </joint>
   <!-- Base Link -->
   <link name="base_link">
@@ -11,5 +18,4 @@
       <origin xyz="0 0 0" rpy="0 0 0"/>
       <geometry>
-        <!-- Assuming a ROS package named 'ceto_description/description' exists -->
         <mesh filename="file://$(find ceto_description)/models/meshes/bluerov2.dae" scale="0.025 0.025 0.025"/>
       </geometry>

Commit message: error repo, two different tfs due to gzbridge tf and urdf tf

File: urdf/robot.urdf.xacro (robot description, xacro)
@@ -2,10 +2,10 @@
 <robot name="ceto">
 <!-- add a dummy root (no inertia) to satisfy KDL -->
-  <link name="root_link"/>
+  <!-- <link name="root_link"/>
   <joint name="root_to_base_fixed" type="fixed">
     <parent link="root_link"/>
     <child link="base_link"/>
     <origin xyz="0 0 0" rpy="0 0 0"/>
-  </joint>
+  </joint> -->
   <!-- Base Link -->
   <link name="base_link">
